File: KiCad/Nexus-AE-PCB/Nexus-AE-PCB-ControlPath.kicad_sch (KiCad schematic)
At the start: 43 parts, among them J7 SD_CONN, U6 MCP6002T-I_MS, U7 USBLC6-2SC6, U8 MCP6002T-I_MS, U9 74xGxx_MDD_74AHCT1G125GV

Commit message: PCB and schmeatic are both approx 90% complete
Parts:
- removed C37: 10nF, Capacitor_SMD:C_0603_1608Metric, symbol Device:C
- removed C38: 1nF, Capacitor_SMD:C_0603_1608Metric, symbol Device:C
- removed C39, C43, C48: 100nF, Capacitor_SMD:C_0603_1608Metric, symbol Device:C
- removed C40: 10uF, Capacitor_SMD:C_0603_1608Metric, symbol Device:C
- removed F1: SMD0603-050, Fuse:Fuse_0603_1608Metric, symbol Device:Polyfuse_Small
- removed J7: SD_CONN, Connector_PinSocket_2.54mm:PinSocket_2x04_P2.54mm_Vertical, symbol Connector_Generic:Conn_02x04_Odd_Even
- removed R64, R67: 56K, Resistor_SMD:R_0603_1608Metric, symbol Device:R_US
- removed R65, R68: 10K, Resistor_SMD:R_0603_1608Metric, symbol Device:R_US
- removed R66: 12.7K, Resistor_SMD:R_0603_1608Metric, symbol Device:R_US
- removed R69: 1K, Resistor_SMD:R_0603_1608Metric, symbol Device:R_US
- removed R70, R71: 100K, Resistor_SMD:R_0603_1608Metric, symbol Device:R_US
- removed R74: 100R, Resistor_SMD:R_0603_1608Metric, symbol Device:R_US
- removed U6: MCP6002T-I_MS, clectric-diy:Amplifier_Operational_Microchip_MCP6002T-I_MS, symbol clectric-diy:Amplifier_Operational_Microchip_MCP6002-xSN
- removed U7: USBLC6-2SC6, Package_TO_SOT_SMD:SOT-23-6, symbol Power_Protection:USBLC6-2SC6
- removed U8: MCP6002T-I_MS, clectric-diy:Amplifier_Operational_Microchip_MCP6002T-I_MS, symbol Amplifier_Operational:MCP6002-xMS
- removed U9: 74xGxx_MDD_74AHCT1G125GV, clectric-diy:74xGxx_MDD_74AHCT1G125GV, symbol clectric-diy:74xGxx_MDD_74AHCT1G125GV
- removed USB1: USB_C_Receptacle_H8.8mm_Jing_918-648K2027E30002, clectric-diy:USB_C_Receptacle_H8.8mm_Jing_918-648K2027E30002, symbol clectric-diy:USB_C_Receptacle_H8.8mm_Jing_918-648K2027E30002
- added J4: AVR-UPDI-6, symbol Connector:AVR-UPDI-6
- C26: renamed from C35; footprint Capacitor_SMD:C_0603_1608Metric -> Capacitor_SMD:C_0402_1005Metric
- C27: renamed from C36; footprint Capacitor_SMD:C_0603_1608Metric -> Capacitor_SMD:C_0402_1005Metric
- C28: renamed from C41; footprint Capacitor_SMD:C_0603_1608Metric -> Capacitor_SMD:C_0402_1005Metric
- C29: renamed from C42; footprint Capacitor_SMD:C_0603_1608Metric -> Capacitor_SMD:C_0402_1005Metric
- C30: renamed from C33; footprint Capacitor_SMD:C_0603_1608Metric -> Capacitor_SMD:C_0402_1005Metric
- C31: renamed from C34; footprint Capacitor_SMD:C_0603_1608Metric -> Capacitor_SMD:C_0402_1005Metric
- C32: renamed from C46; footprint Capacitor_SMD:C_0603_1608Metric -> Capacitor_SMD:C_0402_1005Metric
- C33: renamed from C44; footprint Capacitor_SMD:C_0603_1608Metric -> Capacitor_SMD:C_0402_1005Metric
- C34: renamed from C45; footprint Capacitor_SMD:C_0603_1608Metric -> Capacitor_SMD:C_0402_1005Metric
- C35: renamed from C47; footprint Capacitor_SMD:C_0603_1608Metric -> Capacitor_SMD:C_0402_1005Metric
- D2: renamed from D4; value BAT54S -> BAT54SW; footprint Package_TO_SOT_SMD:SOT-23 -> Package_TO_SOT_SMD:SOT-323_SC-70; symbol Diode:BAT54S -> Diode:BAT54SW
- D3: renamed from D5; value BAT54S -> BAT54SW; footprint Package_TO_SOT_SMD:SOT-23 -> Package_TO_SOT_SMD:SOT-323_SC-70; symbol Diode:BAT54S -> Diode:BAT54SW
- R37: renamed from R55; footprint Resistor_SMD:R_0603_1608Metric -> Resistor_SMD:R_0402_1005Metric
- R38: renamed from R63; footprint Resistor_SMD:R_0603_1608Metric -> Resistor_SMD:R_0402_1005Metric
- R39: renamed from R56; footprint Resistor_SMD:R_0603_1608Metric -> Resistor_SMD:R_0402_1005Metric
- R40: renamed from R53; footprint Resistor_SMD:R_0603_1608Metric -> Resistor_SMD:R_0402_1005Metric
- R41: renamed from R62; footprint Resistor_SMD:R_0603_1608Metric -> Resistor_SMD:R_0402_1005Metric
- R42: renamed from R54; footprint Resistor_SMD:R_0603_1608Metric -> Resistor_SMD:R_0402_1005Metric
- R43: renamed from R72; footprint Resistor_SMD:R_0603_1608Metric -> Resistor_SMD:R_0402_1005Metric
- R44: renamed from R73; footprint Resistor_SMD:R_0603_1608Metric -> Resistor_SMD:R_0402_1005Metric
- R45: renamed from R75; footprint Resistor_SMD:R_0603_1608Metric -> Resistor_SMD:R_0402_1005Metric
Connections:
- no-connect marks 2 -> 0
Other:
- note removed: "MicroSD Card Reader Connector (Reader on Panel)"
- note removed: "USB Host Connector"
- note removed: "Use "Extra" Op Amp to create 2V5 Reference"
